Commit message: Fix.the whole urdf has been wrong axes not aligned causing break , and extra grippers

File: rudra_arm/urdf/rudra_arm1.urdf (robot description, URDF)
Before this commit: robot ARM YPR GRIPPER_7(3), 8 links, 7 joints
Links:
- link base_link: mass 4.02995163253206 -> 4.50779680589233
- link grip: mass 0.0848713844080814 -> 0.134543517946272
- link pitch: mass 0.925309237354222 -> 0.408155014247325
- link pulley: mass 1.78809301817132 -> 1.1765100986821
- link roll: mass 0.82217408126112 -> 0.305019859228966
- link turntable: mass 2.52870378509004 -> 2.52870378509003
- link worm_pitch: mass 3.22088245146418 -> 3.22088245146173
Joints:
- joint grip: axis 0 0 0 -> 0 0 -1; limit (none) -> lower=-3.14 upper=3.14 effort=0 velocity=0; origin xyz=0.026864 -0.025906 -0.17748 rpy=2.3562 1.5708 0 -> xyz=0.086479 -0.086479 -0.11021 rpy=2.3562 -1.5708 0
- joint pitch1_joint: axis 0 0 0 -> -1 0 0; limit lower=0 upper=0 effort=0 velocity=0 -> lower=-3.14 upper=3.14 effort=0 velocity=0; origin xyz=-0.077669 -0.034657 -0.35972 rpy=1.5708 0 1.9905 -> xyz=0.0735164068372525 0.077745638479509 -0.151720000000009 rpy=1.5707963267949 0 0.417471964024542
- joint pitch2_joint: axis 0 0 0 -> 0 0 -1; limit lower=0 upper=0 effort=0 velocity=0 -> lower=-3.14 upper=3.14 effort=0 velocity=0; origin xyz=-0.06 -0.29638 0.3046 rpy=1.5708 -1.3527 -1.5708 -> xyz=-0.0599999999999885 -0.289979355471976 0.310703996433991 rpy=1.5707963267949 -1.37469687411002 -1.5707963267949
- joint roll: axis 0 0 0 -> 0 0 1; limit lower=0 upper=0 effort=0 velocity=0 -> lower=-3.14 upper=3.14 effort=0 velocity=0
- joint turntable_joint: limit lower=0 upper=0 effort=0 velocity=0 -> lower=-3.14 upper=3.14 effort=0 velocity=0; origin xyz=1.3062 -0.008 -0.21244 rpy=1.5708 0.4197 -3.1416 -> xyz=1.35 -0.216 -0.31116 rpy=1.5708 -1.1533 3.1416; type continuous -> revolute
- joint ypr_pitch_joint: axis 0 0 0 -> -1 0 0; limit lower=0 upper=0 effort=0 velocity=0 -> lower=-3.14 upper=3.14 effort=0 velocity=0
