Commit message: feat:successfully loaded and checked motion of rudraas arm

File: rudra_arm/urdf/rudra_arm.urdf (robot description, URDF)
Before this commit: robot ARM YPR GRIPPER_7, 8 links, 7 joints
Links:
- removed link yaw
- added link worldb
- link base_link: geometry collision mesh filename=../meshes/base_link.STL; visual mesh filename=../meshes/base_link.STL
- link grip: geometry collision mesh filename=../meshes/grip.STL; visual mesh filename=../meshes/grip.STL
- link pitch: mass 0.408155013631044 -> 0.408155014247325; geometry collision mesh filename=../meshes/pitch.STL; visual mesh filename=../meshes/pitch.STL
- link pulley: geometry collision mesh filename=../meshes/pulley.STL; visual mesh filename=../meshes/pulley.STL
- link roll: mass 0.830943621943882 -> 0.305019859228966; geometry collision mesh filename=../meshes/roll.STL; visual mesh filename=../meshes/roll.STL
- link turntable: geometry collision mesh filename=../meshes/turntable.STL; visual mesh filename=../meshes/turntable.STL
- link worm_pitch: geometry collision mesh filename=../meshes/worm_pitch.STL; visual mesh filename=../meshes/worm_pitch.STL
Joints:
- removed joint gripper
- removed joint ypr_roll_joint
- removed joint ypr_yaw_joint
- added joint grip: type revolute, parent roll, child grip, origin xyz=0.086479 -0.086479 -0.11021 rpy=2.3562 -1.5708 0, axis 0 0 -1, limit lower=-3.14 upper=3.14 effort=0 velocity=0
- added joint roll: type continuous, parent pitch, child roll, origin xyz=0.05225 0.069756 0 rpy=1.5708 -1.1062 0, axis 0 0 1, limit lower=-3.14 upper=3.14 effort=0 velocity=0
- added joint world_joint: type fixed, parent worldb, child base_link, origin xyz=0 0 0 rpy=-1.5708 0 0
- joint pitch1_joint: axis 0 1 0 -> -1 0 0; limit lower=0 upper=0 effort=0 velocity=0 -> lower=-3.14 upper=3.14 effort=0 velocity=0; type fixed -> revolute
- joint pitch2_joint: axis 0.194845033127278 -0.980834039512103 0 -> 0 0 -1; limit lower=0 upper=0 effort=0 velocity=0 -> lower=-3.14 upper=3.14 effort=0 velocity=0; type fixed -> revolute
- joint turntable_joint: axis 0 0 0 -> 0 0 -1; limit (none) -> lower=-3.14 upper=3.14 effort=0 velocity=0; origin xyz=1.35000046806038 -0.216 -0.311161541452805 rpy=1.5707963267949 -1.15332436277035 3.14159265358979 -> xyz=1.35 -0.216 -0.31116 rpy=1.5708 -1.1533 3.1416; type fixed -> revolute
- joint ypr_pitch_joint: axis 0 0.452902695109985 0.89155995242166 -> -1 0 0; limit lower=0 upper=0 effort=0 velocity=0 -> lower=-3.14 upper=3.14 effort=0 velocity=0; origin xyz=-0.190507127605395 -0.177675757893486 -0.112004491525251 rpy=0.904678468556746 -1.5707963267949 0 -> xyz=-0.19051 -0.17768 -0.112 rpy=0.90468 -1.5708 0; type fixed -> revolute

Commit message: feat:added the base frame to check if collisions occur they do occur

File: rudra_arm/urdf/rudra_arm.urdf (robot description, URDF)
Before this commit: robot ARM YPR GRIPPER_7, 8 links, 7 joints
Links:
- link base_link: geometry collision mesh filename=../meshes/base_link.STL; visual mesh filename=../meshes/base_link.STL

Commit message: Fix.got back the original urdf , checked no mech error , need to check collisions

File: rudra_arm/urdf/rudra_arm.urdf (robot description, URDF)
Before this commit: robot ARM YPR GRIPPER_7, 8 links, 7 joints
Joints:
- joint turntable_joint: origin xyz=1.35 -0.216 -0.31116 rpy=1.5708 -1.1533 3.1416 -> xyz=1.35 -0.216 -0.3112 rpy=1.5708 -1.1533 3.1416

Commit message: feat:rudra arm simulation changed the urdf file for proper gripper orientation and the turntable

File: rudra_arm/urdf/rudra_arm.urdf (robot description, URDF)
Before this commit: robot ARM YPR GRIPPER_7, 8 links, 7 joints
Links:
- link pitch: mass 0.408155014247325 -> 0.925309423783586
- link pulley: mass 1.1765100986821 -> 1.78809248147294
- link roll: mass 0.305019859228966 -> 0.822174268776543
Joints:
- joint pitch2_joint: origin xyz=-0.0599999999999885 -0.289979355471976 0.310703996433991 rpy=1.5707963267949 -1.37469687411002 -1.5707963267949 -> xyz=-0.06 -0.28998 0.3107 rpy=1.5708 -1.3747 -1.5708
- joint roll: axis 0 0 1 -> 0 0 -1
- joint turntable_joint: origin xyz=1.35 -0.216 -0.3112 rpy=1.5708 -1.1533 3.1416 -> xyz=1.35000046806038 -0.216 -0.311161541452805 rpy=1.5707963267949 -1.15332436277035 3.14159265358979

Commit message: feat:changed the arm removed the motor still axis of rotation is there

File: rudra_arm/urdf/rudra_arm.urdf (robot description, URDF)
Before this commit: robot ARM YPR GRIPPER_7, 8 links, 7 joints
Links:
- link base_link: mass 4.50779680589233 -> 4.02995163253206
- link pitch: mass 0.925309423783586 -> 0.925309424196917
- link roll: mass 0.822174268776543 -> 0.687630751243602
Joints:
- joint grip: axis 0 0 -1 -> 0 0 0; limit lower=-3.14 upper=3.14 effort=0 velocity=0 -> lower=0 upper=0 effort=0 velocity=0; type revolute -> fixed
- joint pitch1_joint: limit lower=-3.14 upper=3.14 effort=0 velocity=0 -> lower=0 upper=0 effort=0 velocity=0; origin xyz=0.0735164068372525 0.077745638479509 -0.151720000000009 rpy=1.5707963267949 0 0.417471964024542 -> xyz=0.073516 0.077746 -0.15172 rpy=1.5708 0 0.41747
- joint pitch2_joint: limit lower=-3.14 upper=3.14 effort=0 velocity=0 -> lower=0 upper=0 effort=0 velocity=0
- joint roll: limit lower=-3.14 upper=3.14 effort=0 velocity=0 -> lower=0 upper=0 effort=0 velocity=0
- joint turntable_joint: limit lower=-3.14 upper=3.14 effort=0 velocity=0 -> lower=0 upper=0 effort=0 velocity=0; origin xyz=1.35000046806038 -0.216 -0.311161541452805 rpy=1.5707963267949 -1.15332436277035 3.14159265358979 -> xyz=1.35 -0.216 -0.31116 rpy=1.5708 -1.1533 3.1416
- joint ypr_pitch_joint: limit lower=-3.14 upper=3.14 effort=0 velocity=0 -> lower=0 upper=0 effort=0 velocity=0

Commit message: feat:made changes to make sure the turntable doesnt move not working

File: rudra_arm/urdf/rudra_arm.urdf (robot description, URDF)
Before this commit: robot (3), 8 links, 7 joints
Links:
- removed link grip
- link pitch: mass 0.925309424196917 -> 0.925309312313834
- link pulley: mass 1.78809248147294 -> 1.78809149742768
- link roll: mass 0.687630751243602 -> 0.82217415730679
- link turntable: mass 2.52870378509003 -> 2.52870378509004
- link worm_pitch: mass 3.22088245146173 -> 3.22088245145389
Joints:
- removed joint grip
- joint pitch1_joint: limit lower=0 upper=0 effort=0 velocity=0 -> lower=-3.14 upper=3.14 effort=0 velocity=0; origin xyz=0.073516 0.077746 -0.15172 rpy=1.5708 0 0.41747 -> xyz=0.0735164068372525 0.077745638479509 -0.151720000000009 rpy=1.5707963267949 0 0.417471964024542
- joint pitch2_joint: limit lower=0 upper=0 effort=0 velocity=0 -> lower=-3.14 upper=3.14 effort=0 velocity=0; origin xyz=-0.06 -0.28998 0.3107 rpy=1.5708 -1.3747 -1.5708 -> xyz=-0.0599999999999885 -0.289979355471976 0.310703996433991 rpy=1.5707963267949 -1.37469687411002 -1.5707963267949
- joint roll: axis 0 0 -1 -> -0.57847 -0.28989 -0.76245; limit lower=0 upper=0 effort=0 velocity=0 -> lower=-3.14 upper=3.14 effort=0 velocity=0
- joint turntable_joint: limit lower=0 upper=0 effort=0 velocity=0 -> lower=-3.14 upper=3.14 effort=0 velocity=0; origin xyz=1.35 -0.216 -0.31116 rpy=1.5708 -1.1533 3.1416 -> xyz=1.35000046806038 -0.216 -0.311161541452805 rpy=1.5707963267949 -1.15332436277035 3.14159265358979
- joint ypr_pitch_joint: limit lower=0 upper=0 effort=0 velocity=0 -> lower=-3.14 upper=3.14 effort=0 velocity=0

Commit message: feat:tried to change the urdf model to make it so that the gripper is added (urdf is wrong)

File: rudra_arm/urdf/rudra_arm.urdf (robot description, URDF)
Before this commit: robot ARM YPR GRIPPER_7(2), 7 links, 6 joints
Links:
- added link grip, mass 0.0848713844080814; collision mesh filename=../meshes/grip.STL; visual mesh filename=../meshes/grip.STL
- link pitch: mass 0.925309312313834 -> 0.925309237354222
- link pulley: mass 1.78809149742768 -> 1.78809301817132
- link roll: mass 0.82217415730679 -> 0.82217408126112
- link worm_pitch: mass 3.22088245145389 -> 3.22088245146418
Joints:
- added joint grip: type fixed, parent roll, child grip, origin xyz=0.026864 -0.025906 -0.17748 rpy=2.3562 1.5708 0, axis 0 0 0
- joint pitch1_joint: axis -1 0 0 -> 0 0 0; limit lower=-3.14 upper=3.14 effort=0 velocity=0 -> lower=0 upper=0 effort=0 velocity=0; origin xyz=0.0735164068372525 0.077745638479509 -0.151720000000009 rpy=1.5707963267949 0 0.417471964024542 -> xyz=-0.077669 -0.034657 -0.35972 rpy=1.5708 0 1.9905
- joint pitch2_joint: axis 0 0 -1 -> 0 0 0; limit lower=-3.14 upper=3.14 effort=0 velocity=0 -> lower=0 upper=0 effort=0 velocity=0; origin xyz=-0.0599999999999885 -0.289979355471976 0.310703996433991 rpy=1.5707963267949 -1.37469687411002 -1.5707963267949 -> xyz=-0.06 -0.29638 0.3046 rpy=1.5708 -1.3527 -1.5708
- joint roll: axis -0.57847 -0.28989 -0.76245 -> 0 0 0; limit lower=-3.14 upper=3.14 effort=0 velocity=0 -> lower=0 upper=0 effort=0 velocity=0
- joint turntable_joint: limit lower=-3.14 upper=3.14 effort=0 velocity=0 -> lower=0 upper=0 effort=0 velocity=0; origin xyz=1.35000046806038 -0.216 -0.311161541452805 rpy=1.5707963267949 -1.15332436277035 3.14159265358979 -> xyz=1.3062 -0.008 -0.21244 rpy=1.5708 0.4197 -3.1416; type revolute -> continuous
- joint ypr_pitch_joint: axis -1 0 0 -> 0 0 0; limit lower=-3.14 upper=3.14 effort=0 velocity=0 -> lower=0 upper=0 effort=0 velocity=0

Commit message: Fix.wrong still the turntable is tilted the others are not functioning well

File: rudra_arm/urdf/rudra_arm.urdf (robot description, URDF)
Before this commit: robot ARM YPR GRIPPER_7, 8 links, 7 joints
Links:
- removed link grip
- removed link pitch
- removed link pulley
- removed link roll
- removed link worm_pitch
- added link claw, mass 0.078604; collision mesh filename=../meshes/claw.STL; visual mesh filename=../meshes/claw.STL
- added link diff 2, mass 0.50646; collision mesh filename=../meshes/diff 2.STL; visual mesh filename=../meshes/diff 2.STL
- added link diff1, mass 0.33528; collision mesh filename=../meshes/diff1.STL; visual mesh filename=../meshes/diff1.STL
- added link link1, mass 2.6849; collision mesh filename=../meshes/link1.STL; visual mesh filename=../meshes/link1.STL
- added link link2, mass 1.7567; collision mesh filename=../meshes/link2.STL; visual mesh filename=../meshes/link2.STL
- link base_link: mass 4.50779680589233 -> 4.0876
- link turntable: mass 2.52870378509003 -> 2.5424
Joints:
- removed joint grip
- removed joint pitch1_joint
- removed joint pitch2_joint
- removed joint roll
- removed joint turntable_joint
- removed joint ypr_pitch_joint
- added joint claw: type prismatic, parent diff 2, child claw, origin xyz=0.12531 -0.028177 0.12448 rpy=3.1416 -1.5708 0, axis 0 0 1, limit lower=-3.14 upper=3.14 effort=0 velocity=0
- added joint pitch: type revolute, parent link2, child diff1, origin xyz=-0.22864 -0.20765 -0.10663 rpy=-3.1416 0 -1.75, axis 0 0 1, limit lower=-3.14 upper=3.14 effort=0 velocity=0
- added joint pitch1: type revolute, parent turntable, child link1, origin xyz=0.050075 -0.13572 0.068746 rpy=3.1416 -0.62954 3.1416, axis -1 0 0, limit lower=-3.14 upper=3.14 effort=0 velocity=0
- added joint pitch2: type revolute, parent link1, child link2, origin xyz=-0.081 -0.29511 0.30583 rpy=1.5708 -1.2551 -1.5708, axis 0 0 -1, limit lower=-3.14 upper=3.14 effort=0 velocity=0
- added joint turntable: type revolute, parent base_link, child turntable, origin xyz=1.3062 -0.232 -0.21244 rpy=0 0.94126 0, axis 0 -1 0, limit lower=-6.28 upper=6.28 effort=0 velocity=0
- added joint yprroll: type revolute, parent diff1, child diff 2, origin xyz=0.019826 0.089558 0.048964 rpy=-1.5708 1.25 -0.84529, axis 0 0 1, limit lower=-3.14 upper=3.14 effort=0 velocity=0

Commit message: Fix.made the arm orientatiomn right but link rotation is wrong now

File: rudra_arm/urdf/rudra_arm.urdf (robot description, URDF)
Before this commit: robot ARM urdf, 8 links, 7 joints
Links:
- removed link claw
- removed link diff 2
- removed link diff1
- removed link link1
- removed link link2
- added link grip, mass 0.134543517946272; collision mesh filename=../meshes/grip.STL; visual mesh filename=../meshes/grip.STL
- added link pitch, mass 0.925309423783586; collision mesh filename=../meshes/pitch.STL; visual mesh filename=../meshes/pitch.STL
- added link pulley, mass 1.78809248147294; collision mesh filename=../meshes/pulley.STL; visual mesh filename=../meshes/pulley.STL
- added link roll, mass 0.822174268776543; collision mesh filename=../meshes/roll.STL; visual mesh filename=../meshes/roll.STL
- added link worm_pitch, mass 3.22088245146173; collision mesh filename=../meshes/worm_pitch.STL; visual mesh filename=../meshes/worm_pitch.STL
- link base_link: mass 4.0876 -> 4.50779680589233; geometry collision mesh filename=../meshes/base_link.STL; visual mesh filename=package://ARM YPR GRIPPER_7/meshes/base_link.STL
- link turntable: mass 2.5424 -> 2.52870378509003; geometry collision mesh filename=../meshes/turntable.STL; visual mesh filename=package://ARM YPR GRIPPER_7/meshes/turntable.STL
Joints:
- removed joint claw
- removed joint pitch
- removed joint pitch1
- removed joint pitch2
- removed joint turntable
- removed joint yprroll
- added joint grip: type prismatic, parent roll, child grip, origin xyz=0.086479 -0.086479 -0.11021 rpy=2.3562 -1.5708 0, axis 0 0 -1, limit lower=-3.14 upper=3.14 effort=0 velocity=0
- added joint pitch1_joint: type revolute, parent turntable, child worm_pitch, origin xyz=0.0735164068372525 0.077745638479509 -0.151720000000009 rpy=1.5707963267949 0 0.417471964024542, axis -1 0 0, limit lower=-3.14 upper=3.14 effort=0 velocity=0
- added joint pitch2_joint: type revolute, parent worm_pitch, child pulley, origin xyz=-0.06 -0.28998 0.3107 rpy=1.5708 -1.3747 -1.5708, axis 0 0 -1, limit lower=-3.14 upper=3.14 effort=0 velocity=0
- added joint roll: type continuous, parent pitch, child roll, origin xyz=0.05225 0.069756 0 rpy=1.5708 -1.1062 0, axis 0 0 -1, limit lower=-3.14 upper=3.14 effort=0 velocity=0
- added joint turntable_joint: type revolute, parent base_link, child turntable, origin xyz=1.35000046806038 -0.216 -0.311161541452805 rpy=1.5707963267949 -1.15332436277035 3.14159265358979, axis 0 0 -1, limit lower=-6.28 upper=6.28 effort=0 velocity=0
- added joint ypr_pitch_joint: type revolute, parent pulley, child pitch, origin xyz=-0.19051 -0.17768 -0.112 rpy=0.90468 -1.5708 0, axis -1 0 0, limit lower=-3.14 upper=3.14 effort=0 velocity=0
