Commit message: feat:tried with new urdf arm still same issue base link not attached with turntable

File: rudra_arm/urdf/Assem1.urdf (robot description, URDF)
Before this commit: robot Assem ARM, 6 links, 5 joints
Links:
- removed link diff1
- removed link diff2
- removed link link1
- removed link link2
- removed link turtable
- added link 1st link, mass 1.8407; collision mesh filename=../meshes/1st link.STL; visual mesh filename=../meshes/1st link.STL
- added link 2nd link, mass 0.96031; collision mesh filename=../meshes/2nd link.STL; visual mesh filename=../meshes/2nd link.STL
- added link turntable, mass 1.2414; collision mesh filename=../meshes/turntable.STL; visual mesh filename=../meshes/turntable.STL
- added link ypr pitch, mass 0.21134; collision mesh filename=../meshes/ypr pitch.STL; visual mesh filename=../meshes/ypr pitch.STL
- added link ypr roll, mass 0.68469; collision mesh filename=../meshes/ypr roll.STL; visual mesh filename=../meshes/ypr roll.STL
Joints:
- removed joint pitch1
- removed joint pitch2
- removed joint ypr pitch
- removed joint yprroll
- added joint 1st link: type fixed, parent turntable, child 1st link, origin xyz=0.074167 0.19772 0.041626 rpy=0 0 0, axis 0 0 -1
- added joint 2nd link: type fixed, parent 1st link, child 2nd link, origin xyz=-0.26523 0.29511 -0.1523 rpy=0 0 0, axis 0 0 -1
- added joint pitch: type revolute, parent 2nd link, child ypr pitch, origin xyz=0.22268 0.19482 0.092911 rpy=0 0 0, axis -0.48941 0 0.87205, limit lower=0 upper=0 effort=0 velocity=0
- added joint roll: type revolute, parent ypr pitch, child ypr roll, origin xyz=0.0064818 0.030526 0.033306 rpy=0 0 0, axis 0.50916 0.81185 0.28575, limit lower=0 upper=0 effort=0 velocity=0
- joint turntable: axis 0 0 -1 -> 0 -1 0; child turtable -> turntable; limit lower=-3.14 upper=3.14 effort=0 velocity=0 -> lower=0 upper=0 effort=0 velocity=0; origin xyz=-1.0002 -0.14506 0.0063099 rpy=0 0 -0.012421 -> xyz=0.45345 0.166 0.24526 rpy=0 0 0
