Commit message: feat:made the new arm urdf it is working and staying intact issues with base frame

File: rudra_arm/urdf/rudra_arm_final.urdf (robot description, URDF)
Before this commit: robot N1, 8 links, 7 joints
Links:
- removed link end
- removed link ypr1
- removed link ypr2
- added link claw, mass 0.086144; collision mesh filename=../meshes/claw.STL; visual mesh filename=../meshes/claw.STL
- added link ypr pitch, mass 0.19925; collision mesh filename=../meshes/ypr pitch.STL; visual mesh filename=../meshes/ypr pitch.STL
- added link ypr roll, mass 0.59855; collision mesh filename=../meshes/ypr roll.STL; visual mesh filename=../meshes/ypr roll.STL
- link base_link: mass 12.7671132805366 -> 12.767
- link link1: mass 0.229444432647079 -> 0.22944
- link link2: mass 0.209369199831917 -> 0.20937
- link link3: mass 0.434663057886458 -> 0.43466
- link tt: mass 0.129929642618295 -> 0.12993
Joints:
- removed joint end
- removed joint ypr1
- removed joint ypr2
- added joint claw: type prismatic, parent ypr roll, child claw, origin xyz=-0.00027829 0.08223 -0.11311 rpy=3.1416 -0.34776 -0.032181, axis 0 -1 0, limit lower=-3.14 upper=3.14 effort=0 velocity=0
- added joint ypr pitch: type revolute, parent link3, child ypr pitch, origin xyz=-0.028 -0.077678 0.40923 rpy=-1.5708 -0.13663 1.5708, axis -1 0 0, limit lower=-3.14 upper=3.14 effort=0 velocity=0
- added joint ypr roll: type revolute, parent ypr pitch, child ypr roll, origin xyz=0.025873 -0.021203 -0.0070861 rpy=0.010968 -1.2482 -1.5824, axis 0 0 -1, limit lower=-3.14 upper=3.14 effort=0 velocity=0
- joint link1: axis 0 1 0 -> -1 0 0; origin xyz=-3.4934 0.37744 0.82892 rpy=-2.9337 0.8328 -1.8744 -> xyz=0.033255 0.2121 -0.029851 rpy=0 0.025305 0
- joint link2: axis 0 1 0 -> 1 0 0; origin xyz=-0.1351 0.096831 0.14222 rpy=0.053413 0.57538 -0.25746 -> xyz=-0.062 0.30929 0.39286 rpy=0 0 0
- joint link3: axis 0 1 0 -> -1 0 0; origin xyz=-2.0297 -5.947 3.3406 rpy=1.0874 -1.1611 2.3867 -> xyz=0 0.29017 -0.27532 rpy=3.1416 0 3.1416
- joint tt: axis 0 1 0 -> 0 -1 0; origin xyz=0.40275 0.46108 -0.020796 rpy=1.5708 0 0.020119 -> xyz=0.151 0.010905 -0.0415 rpy=0 0 0

Commit message: feat:made the claw fixed so that it moves with the arm

File: rudra_arm/urdf/rudra_arm_final.urdf (robot description, URDF)
Before this commit: robot New Arm(urdf), 8 links, 7 joints
Joints:
- joint claw: type prismatic -> fixed

Commit message: feat:made the arm direction starught and in terms of matlab issue with base frame

File: rudra_arm/urdf/rudra_arm_final.urdf (robot description, URDF)
Before this commit: robot New Arm(urdf), 8 links, 7 joints
Links:
- added link worldb
Joints:
- added joint world_joint: type fixed, parent worldb, child base_link, origin xyz=0 0 0 rpy=-4.7124 0 0

Commit message: feat:made the arm and base link orientation face the same side

File: rudra_arm/urdf/rudra_arm_final.urdf (robot description, URDF)
Before this commit: robot New Arm(urdf), 9 links, 8 joints
Joints:
- joint tt: origin xyz=0.151 0.010905 -0.0415 rpy=0 0 0 -> xyz=0.151 0.010905 -0.0415 rpy=-3.1416 0 0
- joint world_joint: origin xyz=0 0 0 rpy=-4.7124 0 0 -> xyz=0 0 0 rpy=-1.518 0 0
