Commit message: feat:checked if the new arm is attached to the base frame

File: rudra_arm/urdf/rudra_arm_new.urdf (robot description, URDF)
Before this commit: robot New Arm(urdf), 9 links, 8 joints
Links:
- removed link worldb
- link claw: mass 0.086144 -> 0.0861437294327855
- link link1: mass 0.22944 -> 0.229444432647079
- link link2: mass 0.20937 -> 0.209369199831917
- link link3: mass 0.43466 -> 0.434663057886458
- link ypr pitch: mass 0.19925 -> 0.199246612726693
- link ypr roll: mass 0.59855 -> 0.598549884728632
Joints:
- removed joint world_joint
- joint claw: type fixed -> prismatic
- joint tt: origin xyz=0.151 0.010905 -0.0415 rpy=-3.1416 0 0 -> xyz=0.151 0.010905 -0.0415 rpy=0 0 0

Commit message: feat:made them face the same direction

File: rudra_arm/urdf/rudra_arm_new.urdf (robot description, URDF)
Before this commit: robot New Arm(urdf)2, 8 links, 7 joints
Links:
- added link worldb
Joints:
- added joint world_joint: type fixed, parent worldb, child base_link, origin xyz=0 0 0 rpy=-1.518 0 0
- joint claw: type prismatic -> fixed
- joint tt: origin xyz=0.151 0.010905 -0.0415 rpy=0 0 0 -> xyz=0.151 0.010905 -0.0415 rpy=-3.1416 0 0

Commit message: feat:changed the coordinates of the arm to be above the turntable

File: rudra_arm/urdf/rudra_arm_new.urdf (robot description, URDF)
Before this commit: robot New Arm(urdf)2, 9 links, 8 joints
Joints:
- joint tt: origin xyz=0.151 0.010905 -0.0415 rpy=-3.1416 0 0 -> xyz=1.31 -0.0548 -0.212 rpy=-3.1416 0 0

Commit message: feat:rotated the arm by 90 degrees

File: rudra_arm/urdf/rudra_arm_new.urdf (robot description, URDF)
Before this commit: robot New Arm(urdf)2, 9 links, 8 joints
Joints:
- joint tt: origin xyz=1.31 -0.0548 -0.212 rpy=-3.1416 0 0 -> xyz=1.31 -0.0548 -0.212 rpy=-3.1416 1.5708 0

Commit message: feat:the arm is working in random config attached to the robotic arm gotta add collision checking

File: rudra_arm/urdf/rudra_arm_new.urdf (robot description, URDF)
Before this commit: robot New Arm(urdf)2, 9 links, 8 joints
Joints:
- joint tt: limit lower=-3.14 upper=3.14 effort=0 velocity=0 -> lower=-6.28 upper=6.28 effort=0 velocity=0

Commit message: feat:checked for limits of all jointsusing manual loop not great and accurate

File: rudra_arm/urdf/rudra_arm_new.urdf (robot description, URDF)
Before this commit: robot New Arm(urdf)2, 9 links, 8 joints
Joints:
- joint tt: limit lower=-6.28 upper=6.28 effort=0 velocity=0 -> lower=-3.14 upper=3.14 effort=0 velocity=0
